File: SCH_BRD/uart_pc.sch (EAGLE design)
At the start: 72 parts, among them J4 DM3AT-SF-PEJM5, J5 105017-0001, U1 FT232RQ, X20 AK550/2

Commit message: Work .brd 19/09/17
Connections:
- net N$110: now also D39.2; no longer D39.3
- net N$113: now also D39.3; no longer D39.2
Other:
- moved on the sheet: D39, R97, R98, R99, U$4, U$5, U$6
Changed lines of the file:
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@@
 <instance part="C51" gate="G$1" x="-109.22" y="-27.94"/>
 <instance part="SJ27" gate="G$1" x="-58.42" y="-22.86" rot="MR90"/>
-<instance part="D39" gate="G$1" x="73.66" y="30.48"/>
-<instance part="U$4" gate="G$1" x="55.88" y="2.54"/>
-<instance part="U$5" gate="G$1" x="71.12" y="2.54"/>
-<instance part="U$6" gate="G$1" x="86.36" y="2.54"/>
-<instance part="R97" gate="G$1" x="66.04" y="15.24" rot="R270"/>
-<instance part="R98" gate="G$1" x="73.66" y="15.24" rot="R270"/>
-<instance part="R99" gate="G$1" x="81.28" y="15.24" rot="R270"/>
-<instance part="GND134" gate="1" x="58.42" y="-7.62"/>
-<instance part="GND135" gate="1" x="73.66" y="-7.62"/>
-<instance part="GND136" gate="1" x="88.9" y="-7.62"/>
-<instance part="SUPPLY8" gate="G$1" x="73.66" y="43.18"/>
+<instance part="D39" gate="G$1" x="73.66" y="38.1"/>
+<instance part="U$4" gate="G$1" x="55.88" y="5.08"/>
+<instance part="U$5" gate="G$1" x="71.12" y="5.08"/>
+<instance part="U$6" gate="G$1" x="86.36" y="5.08"/>
+<instance part="R97" gate="G$1" x="66.04" y="17.78" rot="R270"/>
+<instance part="R98" gate="G$1" x="73.66" y="17.78" rot="R270"/>
+<instance part="R99" gate="G$1" x="81.28" y="17.78" rot="R270"/>
+<instance part="GND134" gate="1" x="58.42" y="-5.08"/>
+<instance part="GND135" gate="1" x="73.66" y="-5.08"/>
+<instance part="GND136" gate="1" x="88.9" y="-5.08"/>
+<instance part="SUPPLY8" gate="G$1" x="73.66" y="50.8"/>
 <instance part="S2" gate="G$1" x="-71.12" y="-48.26"/>
 <instance part="LED2" gate="G$1" x="104.14" y="25.4"/>
@@
 <pinref part="U$4" gate="G$1" pin="S"/>
 <pinref part="GND134" gate="1" pin="GND"/>
-<wire x1="58.42" y1="-2.54" x2="58.42" y2="-5.08" width="0.1524" layer="91"/>
+<wire x1="58.42" y1="0" x2="58.42" y2="-2.54" width="0.1524" layer="91"/>
 </segment>
 <segment>
 <pinref part="U$5" gate="G$1" pin="S"/>
 <pinref part="GND135" gate="1" pin="GND"/>
-<wire x1="73.66" y1="-2.54" x2="73.66" y2="-5.08" width="0.1524" layer="91"/>
+<wire x1="73.66" y1="0" x2="73.66" y2="-2.54" width="0.1524" layer="91"/>
 </segment>
 <segment>
 <pinref part="U$6" gate="G$1" pin="S"/>
 <pinref part="GND136" gate="1" pin="GND"/>
-<wire x1="88.9" y1="-2.54" x2="88.9" y2="-5.08" width="0.1524" layer="91"/>
+<wire x1="88.9" y1="0" x2="88.9" y2="-2.54" width="0.1524" layer="91"/>
 </segment>
 <segment>
@@
 <pinref part="D39" gate="G$1" pin="1"/>
 <pinref part="SUPPLY8" gate="G$1" pin="3.3V"/>
-<wire x1="73.66" y1="43.18" x2="73.66" y2="40.64" width="0.1524" layer="91"/>
+<wire x1="73.66" y1="50.8" x2="73.66" y2="48.26" width="0.1524" layer="91"/>
 </segment>
 <segment>
@@
 <pinref part="D39" gate="G$1" pin="4"/>
 <pinref part="R97" gate="G$1" pin="1"/>
-<wire x1="66.04" y1="22.86" x2="66.04" y2="20.32" width="0.1524" layer="91"/>
+<wire x1="66.04" y1="30.48" x2="66.04" y2="22.86" width="0.1524" layer="91"/>
 </segment>
 </net>
 <net name="N$110" class="0">
 <segment>
+<pinref part="R98" gate="G$1" pin="1"/>
+<wire x1="73.66" y1="25.4" x2="73.66" y2="22.86" width="0.1524" layer="91"/>
+<pinref part="D39" gate="G$1" pin="2"/>
+<wire x1="81.28" y1="30.48" x2="78.74" y2="30.48" width="0.1524" layer="91"/>
+<wire x1="78.74" y1="30.48" x2="78.74" y2="25.4" width="0.1524" layer="91"/>
+<wire x1="78.74" y1="25.4" x2="73.66" y2="25.4" width="0.1524" layer="91"/>
+</segment>
+</net>
+<net name="N$113" class="0">
+<segment>
+<pinref part="R99" gate="G$1" pin="1"/>
 <pinref part="D39" gate="G$1" pin="3"/>
-<pinref part="R98" gate="G$1" pin="1"/>
-<wire x1="73.66" y1="22.86" x2="73.66" y2="20.32" width="0.1524" layer="91"/>
-</segment>
-</net>
-<net name="N$113" class="0">
-<segment>
-<pinref part="D39" gate="G$1" pin="2"/>
-<pinref part="R99" gate="G$1" pin="1"/>
-<wire x1="81.28" y1="22.86" x2="81.28" y2="20.32" width="0.1524" layer="91"/>
+<wire x1="73.66" y1="30.48" x2="73.66" y2="27.94" width="0.1524" layer="91"/>
+<wire x1="73.66" y1="27.94" x2="81.28" y2="27.94" width="0.1524" layer="91"/>
+<wire x1="81.28" y1="27.94" x2="81.28" y2="22.86" width="0.1524" layer="91"/>
 </segment>
 </net>
@@
 <segment>
 <pinref part="U$4" gate="G$1" pin="D"/>
-<wire x1="58.42" y1="7.62" x2="58.42" y2="10.16" width="0.1524" layer="91"/>
+<wire x1="58.42" y1="10.16" x2="58.42" y2="12.7" width="0.1524" layer="91"/>
 <pinref part="R97" gate="G$1" pin="2"/>
-<wire x1="58.42" y1="10.16" x2="66.04" y2="10.16" width="0.1524" layer="91"/>
+<wire x1="58.42" y1="12.7" x2="66.04" y2="12.7" width="0.1524" layer="91"/>
 </segment>
 </net>
@@
 <pinref part="U$5" gate="G$1" pin="D"/>
 <pinref part="R98" gate="G$1" pin="2"/>
-<wire x1="73.66" y1="7.62" x2="73.66" y2="10.16" width="0.1524" layer="91"/>
+<wire x1="73.66" y1="10.16" x2="73.66" y2="12.7" width="0.1524" layer="91"/>
 </segment>
 </net>
@@
 <segment>
 <pinref part="U$6" gate="G$1" pin="D"/>
-<wire x1="88.9" y1="7.62" x2="88.9" y2="10.16" width="0.1524" layer="91"/>
+<wire x1="88.9" y1="10.16" x2="88.9" y2="12.7" width="0.1524" layer="91"/>
 <pinref part="R99" gate="G$1" pin="2"/>
-<wire x1="88.9" y1="10.16" x2="81.28" y2="10.16" width="0.1524" layer="91"/>
+<wire x1="88.9" y1="12.7" x2="81.28" y2="12.7" width="0.1524" layer="91"/>
 </segment>
 </net>
@@
 <segment>
 <pinref part="U$6" gate="G$1" pin="G"/>
-<wire x1="83.82" y1="0" x2="81.28" y2="0" width="0.1524" layer="91"/>
-<label x="81.28" y="0" size="1.27" layer="95" rot="R180" xref="yes"/>
+<wire x1="83.82" y1="2.54" x2="81.28" y2="2.54" width="0.1524" layer="91"/>
+<label x="81.28" y="2.54" size="1.27" layer="95" rot="R180" xref="yes"/>
 </segment>
 </net>
@@
 <segment>
 <pinref part="U$5" gate="G$1" pin="G"/>
-<wire x1="68.58" y1="0" x2="66.04" y2="0" width="0.1524" layer="91"/>
-<label x="66.04" y="0" size="1.27" layer="95" rot="R180" xref="yes"/>
+<wire x1="68.58" y1="2.54" x2="66.04" y2="2.54" width="0.1524" layer="91"/>
+<label x="66.04" y="2.54" size="1.27" layer="95" rot="R180" xref="yes"/>
 </segment>
 </net>
@@
 <segment>
 <pinref part="U$4" gate="G$1" pin="G"/>
-<wire x1="53.34" y1="0" x2="50.8" y2="0" width="0.1524" layer="91"/>
-<label x="50.8" y="0" size="1.27" layer="95" rot="R180" xref="yes"/>
-</segment>
-</net>
+<wire x1="53.34" y1="2.54" x2="50.8" y2="2.54" width="0.1524" layer="91"/>
+<label x="50.8" y="2.54" size="1.27" layer="95" rot="R180" xref="yes"/>
+</segment>
+</net>

Commit message: Work .brd 20/09/17
Parts:
- removed SJ27: (no value), microbuilder:SOLDERJUMPER_2WAY
- added SVBAT: (no value), SparkFun-Electromechanical:SWITCH-SPDTSMD
- renumbered S3 to S3.3V, S4 to S5V
Connections:
- removed net N$110: D39.2, R98.1
- removed net N$113: D39.3, R99.1
- new net N$11: D39.3, R98.1
- new net N$12: D39.2, R99.1
- net 3.3V: now also SVBAT.S; no longer SJ27.3
- net 3V3OUT: now also S3.3V.S; no longer S3.3V.O
- net 5VOUT: now also S5V.S; no longer S5V.O
- net BAT: now also SVBAT.O; no longer SJ27.1
- net VBAT: now also SVBAT.P; no longer SJ27.2
- net VIN3V3: now also S3.3V.O; no longer S3.3V.S
- net VIN5V: now also S5V.O; no longer S5V.S
Other:
- moved on the sheet: C47
