File: SCH_BRD/uart_pc.brd (EAGLE design)
At the start: 40.6 x 40.6 mm, 72 parts, among them J4 DM3AT-SF-PEJM5, J5 105017-0001, U1 FT232RQ, X20 AK550/2

Commit message: Work .brd 19/09/17
Parts:
- moved U$5 87.0 mm to (-16.6, 44.9)
- moved R98 85.4 mm to (-16.6, 47.7)
- moved C47 83.9 mm to (72.3, 18.2)
- moved C46 83.9 mm to (71.7, 2.92)
- moved U$4 80.8 mm to (-19.7, 44.9)
- moved U$6 80.8 mm to (-13.5, 44.9)
- moved L1 78.9 mm to (70.6, 6.07)
- moved D39 78.7 mm to (-16.6, 45.6), turned to 180 degrees
- moved R97 78.2 mm to (-19.7, 47.7)
- moved SJ27 77.8 mm to (73.6, 14.6)
- moved R99 77.6 mm to (-13.5, 47.7)
- moved R44 75.1 mm to (60.9, 8.08)
- moved LED1 62.3 mm to (21.9, 3.02), turned to 270 degrees
- moved C6 60.2 mm to (18.8, 3.66)
- moved R3 56.9 mm to (25.3, 3.58), turned to 90 degrees
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Connections:
- net N$110: now also D39.2; no longer D39.3
- net N$113: now also D39.3; no longer D39.2
Routing:
- net OSC_OUT: track 6.61 -> 14.9 mm
- net OSC32_IN: track 5.02 -> 12.6 mm
- net OSC_IN: track 6.64 -> 14.0 mm
- net VIN3V3: track 0.00 -> 6.75 mm, vias 0 -> 1
- net N$113: track 0.00 -> 6.58 mm, vias 0 -> 1
- net VIN5V: track 0.00 -> 6.32 mm
- net OSC32_OUT: track 5.02 -> 11.2 mm
- net N$108: track 0.00 -> 5.41 mm, vias 0 -> 1
- net N$110: track 0.00 -> 3.51 mm, vias 0 -> 1
- net N$51: track 0.00 -> 2.80 mm, vias 0 -> 1
- net N$49: track 0.00 -> 2.09 mm, vias 0 -> 1
- net N$126: track 0.00 -> 2.09 mm
- net N$122: track 0.00 -> 2.09 mm
- net N$117: track 0.00 -> 2.09 mm
- net N$3: track 0.00 -> 1.42 mm, vias 0 -> 1
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
Commit message: Work .brd 20/09/17
Parts:
- removed S3, S4: (no value), SparkFun-Electromechanical:AYZ0202
- removed SJ27: (no value), microbuilder:SOLDERJUMPER_2WAY_OPEN_NOPASTE
- added S3.3V, S5V, SVBAT: (no value), SparkFun-Electromechanical:AYZ0202
- moved C47 62.4 mm to (11.0, 29.9), turned to 90 degrees
- moved C46 62.3 mm to (10.1, 12.5), turned to 180 degrees
- moved L1 61.0 mm to (10.1, 14.1)
- moved C38 57.7 mm to (16.8, 16.1)
- moved C40 53.8 mm to (15.2, 19.2)
- moved R44 53.1 mm to (12.7, 30.3), turned to 270 degrees
- moved C39 50.0 mm to (18.3, 19.2), turned to 180 degrees
- moved C42 48.8 mm to (18.3, 17.7), turned to 180 degrees
- moved R18 46.7 mm to (28.4, 19.1), flipped to the top
- moved C43 46.6 mm to (15.2, 17.7)
- moved C44 46.3 mm to (15.2, 20.8)
- moved C41 45.7 mm to (18.3, 20.8), turned to 180 degrees
- moved C17 45.1 mm to (23.2, 21.8), turned to 180 degrees
- moved R19 44.8 mm to (28.4, 17.4), flipped to the top
- moved R26 43.9 mm to (28.4, 20.7), flipped to the top
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Connections:
- removed net N$110: D39.2, R98.1
- removed net N$113: D39.3, R99.1
- new net N$11: D39.3, R98.1
- new net N$12: D39.2, R99.1
- net 3.3V: now also S3.3V.2, SVBAT.3; no longer S3.2, SJ27.3
- net 3V3OUT: now also S3.3V.3; no longer S3.1
- net 5V: now also S5V.2; no longer S4.2
- net 5VOUT: now also S5V.3; no longer S4.1
- net BAT: now also SVBAT.1; no longer SJ27.1
- net VBAT: now also SVBAT.2; no longer SJ27.2
- net VIN3V3: now also S3.3V.1; no longer S3.3
- net VIN5V: now also S5V.1; no longer S4.3
Routing:
- net 3.3V: track 1.04 -> 131.2 mm, vias 1 -> 5
- net VIN3V3: track 6.75 -> 46.9 mm, vias 1 -> 2
- net VIN5V: track 6.32 -> 39.7 mm, vias 0 -> 1
- net NRST: track 0.00 -> 27.8 mm, vias 0 -> 2
- net SDIO.CD: track 0.00 -> 25.1 mm, vias 0 -> 1
- net SDIO.D2: track 0.00 -> 21.0 mm, vias 0 -> 1
- net SDIO.D3: track 0.00 -> 20.2 mm, vias 0 -> 1
- net SDIO.CMD: track 0.00 -> 18.5 mm, vias 0 -> 1
- net VBAT: track 0.00 -> 17.7 mm, vias 0 -> 2
- net BAT: track 0.00 -> 17.6 mm, vias 0 -> 1
- net SWDIO: track 0.00 -> 17.4 mm
- net SDIO.CK: track 0.00 -> 16.8 mm, vias 0 -> 1
- net SWCLK: track 0.00 -> 16.3 mm
- net USART6.TX: track 0.00 -> 14.3 mm
- net SDIO.D0: track 0.00 -> 12.4 mm, vias 0 -> 1
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Other:
- board size 40.6 x 40.6 mm -> 33.5 x 40.6 mm

Commit message: Finished sch and brd
Version beta
Parts:
- moved R2 4.79 mm to (23.2, 2.90), turned to 180 degrees
- moved R1 3.42 mm to (26.8, 2.90)
- moved R4 1.95 mm to (25.0, 13.3)
- moved R3 1.79 mm to (26.2, 11.4)
- moved C2 1.54 mm to (13.1, 2.84)
- moved C5 1.42 mm to (13.1, 4.47), turned to 180 degrees
- moved C6 0.97 mm to (23.1, 8.13)
- moved C51 0.95 mm to (22.6, 17.6)
- moved LED1 0.74 mm to (26.8, 2.90)
- moved U1 0.43 mm to (25.0, 10.2)
- moved C47 0.33 mm to (11.0, 30.3)
- moved LED5 0.28 mm to (23.2, 2.90), turned to 270 degrees
Routing:
- net N$2: track 0.00 -> 24.5 mm, vias 0 -> 2
- net USART3.RX: track 0.00 -> 22.0 mm, vias 0 -> 1
- net N$1: track 0.00 -> 19.5 mm, vias 0 -> 2
- net USART3.TX: track 6.31 -> 23.1 mm, vias 0 -> 1
- net 5V: track 0.00 -> 16.4 mm
- net USART2.RX: track 1.16 -> 16.8 mm
- net USART2.TX: track 1.16 -> 15.4 mm
- net 3.3V: track 131.2 -> 142.5 mm, vias 5 -> 7
- net N$47: track 0.92 -> 5.63 mm
- net VCAP_1: track 0.00 -> 4.69 mm, vias 0 -> 1
- net N$4: track 0.00 -> 3.97 mm, vias 0 -> 1
- net N$6: track 0.00 -> 3.57 mm
- net N$5: track 0.00 -> 3.03 mm
- net N$10: track 0.00 -> 2.40 mm, vias 0 -> 1
- net N$9: track 0.00 -> 2.40 mm, vias 0 -> 1
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Other:
- board text added: "/home/duver/Documents/other/logo vettoriale.bmp"
